Commit message: Phase B1: move link2_to_link3 from mock_arm to real_arm
Joint link2_to_link3 now backed by mycobot_csv plugin slave_index=2
(real EtherCAT drive) instead of mock_components/GenericSystem.

Co-Authored-By: Claude Opus 4.7 (1M context) <noreply@anthropic.com>

File: src/mycobot_ros2/mycobot_moveit_config/config/mycobot_280.ros2_control.xacro (robot description, xacro)
@@ -26,4 +26,16 @@
                 <state_interface name="velocity"/>
             </joint>
+            <joint name="link2_to_link3">
+                <param name="slave_index">2</param>
+                <param name="counts_per_rad">2085932.0</param>
+                <command_interface name="velocity">
+                    <param name="min">-2.0</param>
+                    <param name="max"> 2.0</param>
+                </command_interface>
+                <state_interface name="position">
+                    <param name="initial_value">${initial_positions['link2_to_link3']}</param>
+                </state_interface>
+                <state_interface name="velocity"/>
+            </joint>
         </ros2_control>
         <!-- ============================================================
@@ -44,13 +56,4 @@
                 <param name="calculate_dynamics">true</param>
             </hardware>
-            <joint name="link2_to_link3">
-                <command_interface name="velocity">
-                    <param name="initial_value">0.0</param>
-                </command_interface>
-                <state_interface name="position">
-                    <param name="initial_value">${initial_positions['link2_to_link3']}</param>
-                </state_interface>
-                <state_interface name="velocity"/>
-            </joint>
             <joint name="link3_to_link4">
                 <command_interface name="velocity">
