Commit message: Phase C: move link3_to_link4 to real_arm + gentle gains

File: src/mycobot_ros2/mycobot_moveit_config/config/mycobot_280.ros2_control.xacro (robot description, xacro)
@@ -38,4 +38,16 @@
                 <state_interface name="velocity"/>
             </joint>
+            <joint name="link3_to_link4">
+                <param name="slave_index">3</param>
+                <param name="counts_per_rad">2085932.0</param>
+                <command_interface name="velocity">
+                    <param name="min">-2.0</param>
+                    <param name="max"> 2.0</param>
+                </command_interface>
+                <state_interface name="position">
+                    <param name="initial_value">${initial_positions['link3_to_link4']}</param>
+                </state_interface>
+                <state_interface name="velocity"/>
+            </joint>
         </ros2_control>
         <!-- ============================================================
@@ -56,13 +68,4 @@
                 <param name="calculate_dynamics">true</param>
             </hardware>
-            <joint name="link3_to_link4">
-                <command_interface name="velocity">
-                    <param name="initial_value">0.0</param>
-                </command_interface>
-                <state_interface name="position">
-                    <param name="initial_value">${initial_positions['link3_to_link4']}</param>
-                </state_interface>
-                <state_interface name="velocity"/>
-            </joint>
             <joint name="link4_to_link5">
                 <command_interface name="velocity">

Commit message: joint 4 verified but slave 2 has some hardware errors

File: src/mycobot_ros2/mycobot_moveit_config/config/mycobot_280.ros2_control.xacro (robot description, xacro)
@@ -50,4 +50,16 @@
                 <state_interface name="velocity"/>
             </joint>
+            <joint name="link4_to_link5">
+                <param name="slave_index">4</param>
+                <param name="counts_per_rad">2085932.0</param>
+                <command_interface name="velocity">
+                    <param name="min">-2.0</param>
+                    <param name="max"> 2.0</param>
+                </command_interface>
+                <state_interface name="position">
+                    <param name="initial_value">${initial_positions['link4_to_link5']}</param>
+                </state_interface>
+                <state_interface name="velocity"/>
+            </joint>
         </ros2_control>
         <!-- ============================================================
@@ -68,13 +80,4 @@
                 <param name="calculate_dynamics">true</param>
             </hardware>
-            <joint name="link4_to_link5">
-                <command_interface name="velocity">
-                    <param name="initial_value">0.0</param>
-                </command_interface>
-                <state_interface name="position">
-                    <param name="initial_value">${initial_positions['link4_to_link5']}</param>
-                </state_interface>
-                <state_interface name="velocity"/>
-            </joint>
             <joint name="link5_to_link6">
                 <command_interface name="velocity">

Commit message: made slave 2 mock because it has entered error state

File: src/mycobot_ros2/mycobot_moveit_config/config/mycobot_280.ros2_control.xacro (robot description, xacro)
@@ -4,6 +4,12 @@
         <xacro:property name="initial_positions" value="${xacro.load_yaml(initial_positions_file)['initial_positions']}"/>
         <!-- ============================================================
-             Hardware Block 1: Real EtherCAT drive on joint 1 (slave 1)
-             Uses the verified mycobot_csv plugin in CSV (velocity) mode.
+             Hardware Block 1: Real EtherCAT drives on joints 1, 3, 4
+             (slaves 1, 3, 4). Slave 2 is on the bus but its drive has a
+             persistent vendor-specific fault (0x603F=0x002E, encoder
+             multi-turn-lost) that the firmware doesn't expose a clear
+             SDO for — link2_to_link3 is therefore handled by the mock
+             block below. When slave 2 is recovered (vendor configurator
+             or encoder battery replacement), move link2_to_link3 back
+             into this block.
              ============================================================ -->
         <ros2_control name="${name}_real_arm" type="system">
@@ -12,5 +18,5 @@
                 <!-- EDIT: change ifname to your EtherCAT interface
                      (run `ip link` to find it; commonly enxNNN... for USB-Eth) -->
-                <param name="ifname">enxc8a3623069bf</param>
+                <param name="ifname">enxc817f55f06f6</param>
             </hardware>
             <joint name="link1_to_link2">
@@ -23,16 +29,4 @@
                 <state_interface name="position">
                     <param name="initial_value">${initial_positions['link1_to_link2']}</param>
-                </state_interface>
-                <state_interface name="velocity"/>
-            </joint>
-            <joint name="link2_to_link3">
-                <param name="slave_index">2</param>
-                <param name="counts_per_rad">2085932.0</param>
-                <command_interface name="velocity">
-                    <param name="min">-2.0</param>
-                    <param name="max"> 2.0</param>
-                </command_interface>
-                <state_interface name="position">
-                    <param name="initial_value">${initial_positions['link2_to_link3']}</param>
                 </state_interface>
                 <state_interface name="velocity"/>
@@ -64,5 +58,5 @@
         </ros2_control>
         <!-- ============================================================
-             Hardware Block 2: Mock joints 2-6 + gripper
+             Hardware Block 2: Mock joints 2, 5, 6 + gripper
              mock_components/GenericSystem echoes commands as state, so
              these joints "track" perfectly without real hardware.
@@ -72,4 +66,6 @@
              initial_value on each command_interface prevents NaN states
              at activation when calculate_dynamics integrates the buffer.
+             link2_to_link3 is here only because slave 2 is faulted
+             (see Block 1 header) — move it back to Block 1 once recovered.
              ============================================================ -->
         <ros2_control name="${name}_mock_arm" type="system">
@@ -80,4 +76,13 @@
                 <param name="calculate_dynamics">true</param>
             </hardware>
+            <joint name="link2_to_link3">
+                <command_interface name="velocity">
+                    <param name="initial_value">0.0</param>
+                </command_interface>
+                <state_interface name="position">
+                    <param name="initial_value">${initial_positions['link2_to_link3']}</param>
+                </state_interface>
+                <state_interface name="velocity"/>
+            </joint>
             <joint name="link5_to_link6">
                 <command_interface name="velocity">

Commit message: Re-integrate slave 2 after fault cleared
Slave 2's vendor fault is gone, so move link2_to_link3 back to the
real_arm block and drop the WORKAROUND-SLAVE2 blocks in mycobot_csv
(extra-slave PO2SOconfig + size adjustment). Verified end-to-end:
all 4 drives reach OPERATION_ENABLED and arm_controller reports
"Goal reached, success!" on a MoveIt trajectory. NIC ifname also
updated to enx00e04c360d9d for the current USB-Eth adapter.

counts_per_rad for slave 2 still uses the placeholder 2085932.0;
calibration is tracked separately.

File: src/mycobot_ros2/mycobot_moveit_config/config/mycobot_280.ros2_control.xacro (robot description, xacro)
@@ -4,12 +4,6 @@
         <xacro:property name="initial_positions" value="${xacro.load_yaml(initial_positions_file)['initial_positions']}"/>
         <!-- ============================================================
-             Hardware Block 1: Real EtherCAT drives on joints 1, 3, 4
-             (slaves 1, 3, 4). Slave 2 is on the bus but its drive has a
-             persistent vendor-specific fault (0x603F=0x002E, encoder
-             multi-turn-lost) that the firmware doesn't expose a clear
-             SDO for — link2_to_link3 is therefore handled by the mock
-             block below. When slave 2 is recovered (vendor configurator
-             or encoder battery replacement), move link2_to_link3 back
-             into this block.
+             Hardware Block 1: Real EtherCAT drives on joints 1–4
+             (slaves 1–4).
              ============================================================ -->
         <ros2_control name="${name}_real_arm" type="system">
@@ -18,5 +12,5 @@
                 <!-- EDIT: change ifname to your EtherCAT interface
                      (run `ip link` to find it; commonly enxNNN... for USB-Eth) -->
-                <param name="ifname">enxc817f55f06f6</param>
+                <param name="ifname">enx00e04c360d9d</param>
             </hardware>
             <joint name="link1_to_link2">
@@ -29,4 +23,16 @@
                 <state_interface name="position">
                     <param name="initial_value">${initial_positions['link1_to_link2']}</param>
+                </state_interface>
+                <state_interface name="velocity"/>
+            </joint>
+            <joint name="link2_to_link3">
+                <param name="slave_index">2</param>
+                <param name="counts_per_rad">2085932.0</param>
+                <command_interface name="velocity">
+                    <param name="min">-2.0</param>
+                    <param name="max"> 2.0</param>
+                </command_interface>
+                <state_interface name="position">
+                    <param name="initial_value">${initial_positions['link2_to_link3']}</param>
                 </state_interface>
                 <state_interface name="velocity"/>
@@ -58,5 +64,5 @@
         </ros2_control>
         <!-- ============================================================
-             Hardware Block 2: Mock joints 2, 5, 6 + gripper
+             Hardware Block 2: Mock joints 5, 6 + gripper
              mock_components/GenericSystem echoes commands as state, so
              these joints "track" perfectly without real hardware.
@@ -66,6 +72,4 @@
              initial_value on each command_interface prevents NaN states
              at activation when calculate_dynamics integrates the buffer.
-             link2_to_link3 is here only because slave 2 is faulted
-             (see Block 1 header) — move it back to Block 1 once recovered.
              ============================================================ -->
         <ros2_control name="${name}_mock_arm" type="system">
@@ -76,13 +80,4 @@
                 <param name="calculate_dynamics">true</param>
             </hardware>
-            <joint name="link2_to_link3">
-                <command_interface name="velocity">
-                    <param name="initial_value">0.0</param>
-                </command_interface>
-                <state_interface name="position">
-                    <param name="initial_value">${initial_positions['link2_to_link3']}</param>
-                </state_interface>
-                <state_interface name="velocity"/>
-            </joint>
             <joint name="link5_to_link6">
                 <command_interface name="velocity">

Commit message: MoveIt: promote link5_to_link6 to real EtherCAT (slave 5)
The wrist roll motor was rewired into position 5 on the EtherCAT
daisy-chain alongside the new big motors at slaves 2-3. Move
link5_to_link6 from the mock_arm block into real_arm so the
joint_trajectory_controller drives slave 5 directly. link6_to_link6flange
stays mocked — slave 6 is not yet connected to the bus (5-DOF testing
phase).

Slave→joint mapping is now slaves 1-3 = big base/shoulder/elbow,
slaves 4-5 = small wrist motors. Same counts_per_rad (2085932.0)
applies across both motor types per empirical sweep.

File: src/mycobot_ros2/mycobot_moveit_config/config/mycobot_280.ros2_control.xacro (robot description, xacro)
@@ -4,6 +4,9 @@
         <xacro:property name="initial_positions" value="${xacro.load_yaml(initial_positions_file)['initial_positions']}"/>
         <!-- ============================================================
-             Hardware Block 1: Real EtherCAT drives on joints 1–4
-             (slaves 1–4).
+             Hardware Block 1: Real EtherCAT drives on joints 1–5
+             (slaves 1–5). Slaves 1–3 are big motors (1650 mN·m rated),
+             slaves 4–5 are small wrist motors (200 mN·m rated).
+             Slave 6 (joint 6) is not yet wired; link6_to_link6flange
+             stays mocked below.
              ============================================================ -->
         <ros2_control name="${name}_real_arm" type="system">
@@ -62,7 +65,19 @@
                 <state_interface name="velocity"/>
             </joint>
+            <joint name="link5_to_link6">
+                <param name="slave_index">5</param>
+                <param name="counts_per_rad">2085932.0</param>
+                <command_interface name="velocity">
+                    <param name="min">-2.0</param>
+                    <param name="max"> 2.0</param>
+                </command_interface>
+                <state_interface name="position">
+                    <param name="initial_value">${initial_positions['link5_to_link6']}</param>
+                </state_interface>
+                <state_interface name="velocity"/>
+            </joint>
         </ros2_control>
         <!-- ============================================================
-             Hardware Block 2: Mock joints 5, 6 + gripper
+             Hardware Block 2: Mock joint 6 + gripper
              mock_components/GenericSystem echoes commands as state, so
              these joints "track" perfectly without real hardware.
@@ -80,13 +95,4 @@
                 <param name="calculate_dynamics">true</param>
             </hardware>
-            <joint name="link5_to_link6">
-                <command_interface name="velocity">
-                    <param name="initial_value">0.0</param>
-                </command_interface>
-                <state_interface name="position">
-                    <param name="initial_value">${initial_positions['link5_to_link6']}</param>
-                </state_interface>
-                <state_interface name="velocity"/>
-            </joint>
             <joint name="link6_to_link6flange">
                 <command_interface name="velocity">
